Commit message: commit

File: description/ros2_control.xacro (robot description, xacro)
@@ -2,5 +2,33 @@
 <robot xmlns:xacro="http://www.ros.org/wiki/xacro">
 <!-- HARDWARE INTERFACE FOR THE ROS2 CONTROL MANAGER-->
-    <ros2_control name="GazeboSystem" type="system">
+    <ros2_control name="RealRobot" type="system">
+        <hardware>
+            <plugin>diffdrive_arduino/DiffDriveArduino</plugin>
+                <param name="left_wheel_name">left_wheel_joint</param>
+                <param name="right_wheel_name">right_wheel_joint</param>
+                <param name="loop_rate">30</param>
+                <param name="device">/dev/ttyACM0</param>
+                <param name="baud_rate">9600</param>
+                <param name="timeout">1000</param>
+                <param name="enc_counts_per_rev">80</param>
+        </hardware>
+        <joint name="left_wheel_joint">
+            <command_interface name="velocity">
+                <param name="min">-10</param>
+                <param name="max">10</param>
+            </command_interface>
+            <state_interface name="velocity"/>
+            <state_interface name="position"/>
+        </joint>
+        <joint name="right_wheel_joint">
+            <command_interface name="velocity">
+                <param name="min">-10</param>
+                <param name="max">10</param>
+            </command_interface>
+            <state_interface name="velocity"/>
+            <state_interface name="position"/>
+        </joint>
+    </ros2_control>
+<!--    <ros2_control name="GazeboSystem" type="system">
         <hardware>
             <plugin>gazebo_ros2_control/GazeboSystem</plugin>
@@ -22,5 +50,5 @@
             <state_interface name="position"/>
         </joint>
-    </ros2_control>
+    </ros2_control> -->
 <!-- GAZEBO PLUGIN FOR THE ROS2 CONTROL MANAGER-->
     <gazebo>
